File: hardware/jig/bottom/Step-to-Talk V2 Jig BOTTOM.brd (EAGLE design)
At the start: 41.9 x 36.8 mm, 6 parts

Commit message: Update jig boards for printing.
Routing:
- net MOSI: track 32.4 -> 34.1 mm
