File: hardware/board/Step-to-TalkV2.brd (EAGLE design)
At the start: 20.5 x 24.5 mm, 19 parts, among them J1 Pogo Pad, J2 Pogo Pad, J3 Pogo Pad, J4 Pogo Pad, J5 Pogo Pad, J6 Pogo Pad, U1 ATTINY85

Commit message: Updated V2.1 board with removed thermals, vias on USB connector pads.
Routing:
- net GND: vias 1 -> 3
- added copper zone on layer 16, net GND
Changed lines of the file:
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@@
 <?xml version="1.0" encoding="utf-8"?>
 <!DOCTYPE eagle SYSTEM "eagle.dtd">
-<eagle version="8.2.2">
+<eagle version="9.6.2">
 <drawing>
 <settings>
-<setting alwaysvectorfont="no"/>
+<setting alwaysvectorfont="yes"/>
+<setting keepoldvectorfont="yes"/>
 <setting verticaltext="up"/>
 </settings>
@@
 <layers>
 <layer number="1" name="Top" color="4" fill="1" visible="yes" active="yes"/>
-<layer number="16" name="Bottom" color="1" fill="1" visible="yes" active="yes"/>
+<layer number="16" name="Bottom" color="1" fill="1" visible="no" active="yes"/>
 <layer number="17" name="Pads" color="2" fill="1" visible="yes" active="yes"/>
 <layer number="18" name="Vias" color="2" fill="1" visible="yes" active="yes"/>
@@
 <layer number="20" name="Dimension" color="15" fill="1" visible="yes" active="yes"/>
 <layer number="21" name="tPlace" color="7" fill="1" visible="yes" active="yes"/>
-<layer number="22" name="bPlace" color="7" fill="1" visible="yes" active="yes"/>
+<layer number="22" name="bPlace" color="7" fill="1" visible="no" active="yes"/>
 <layer number="23" name="tOrigins" color="15" fill="1" visible="yes" active="yes"/>
-<layer number="24" name="bOrigins" color="15" fill="1" visible="yes" active="yes"/>
+<layer number="24" name="bOrigins" color="15" fill="1" visible="no" active="yes"/>
 <layer number="25" name="tNames" color="7" fill="1" visible="yes" active="yes"/>
-<layer number="26" name="bNames" color="7" fill="1" visible="yes" active="yes"/>
-<layer number="27" name="tValues" color="7" fill="1" visible="yes" active="yes"/>
-<layer number="28" name="bValues" color="7" fill="1" visible="yes" active="yes"/>
-<layer number="29" name="tStop" color="7" fill="3" visible="yes" active="yes"/>
-<layer number="30" name="bStop" color="7" fill="6" visible="yes" active="yes"/>
+<layer number="26" name="bNames" color="7" fill="1" visible="no" active="yes"/>
+<layer number="27" name="tValues" color="7" fill="1" visible="no" active="yes"/>
+<layer number="28" name="bValues" color="7" fill="1" visible="no" active="yes"/>
+<layer number="29" name="tStop" color="7" fill="3" visible="no" active="yes"/>
+<layer number="30" name="bStop" color="7" fill="6" visible="no" active="yes"/>
 <layer number="31" name="tCream" color="7" fill="4" visible="no" active="yes"/>
 <layer number="32" name="bCream" color="7" fill="5" visible="no" active="yes"/>
@@
 <layer number="37" name="tTest" color="7" fill="1" visible="no" active="yes"/>
 <layer number="38" name="bTest" color="7" fill="1" visible="no" active="yes"/>
-<layer number="39" name="tKeepout" color="4" fill="11" visible="no" active="yes"/>
+<layer number="39" name="tKeepout" color="4" fill="11" visible="yes" active="yes"/>
 <layer number="40" name="bKeepout" color="1" fill="11" visible="no" active="yes"/>
-<layer number="41" name="tRestrict" color="4" fill="10" visible="no" active="yes"/>
+<layer number="41" name="tRestrict" color="4" fill="10" visible="yes" active="yes"/>
 <layer number="42" name="bRestrict" color="1" fill="10" visible="no" active="yes"/>
 <layer number="43" name="vRestrict" color="2" fill="10" visible="no" active="yes"/>
@@
 <layer number="49" name="Reference" color="7" fill="1" visible="no" active="yes"/>
 <layer number="50" name="dxf" color="7" fill="1" visible="no" active="no"/>
-<layer number="51" name="tDocu" color="7" fill="1" visible="no" active="yes"/>
+<layer number="51" name="tDocu" color="7" fill="1" visible="yes" active="yes"/>
 <layer number="52" name="bDocu" color="7" fill="1" visible="no" active="yes"/>
 <layer number="53" name="tGND_GNDA" color="7" fill="9" visible="no" active="no"/>
@@
 <param name="dpMaxLengthDifference" value="10mm"/>
 <param name="dpGapFactor" value="2.5"/>
-<param name="checkGrid" value="0"/>
 <param name="checkAngle" value="0"/>
 <param name="checkFont" value="1"/>
 <param name="checkRestrict" value="1"/>
+<param name="checkStop" value="0"/>
+<param name="checkValues" value="0"/>
+<param name="checkNames" value="1"/>
+<param name="checkWireStubs" value="1"/>
+<param name="checkPolygonWidth" value="0"/>
 <param name="useDiameter" value="13"/>
 <param name="maxErrors" value="50"/>
@@
 <attribute name="VALUE" x="11.25" y="23.25" size="1.27" layer="27" rot="R270"/>
 </element>
-<element name="H2" library="holes" library_urn="urn:adsk.eagle:library:237" package="4,3-PAD" value="Mounting Pad" x="7.5" y="6"/>
-<element name="J1" library="SparkFun-Connectors" package="PAD.03X.03" value="Pogo Pad" x="16" y="23" rot="MR0"/>
-<element name="J2" library="SparkFun-Connectors" package="PAD.03X.03" value="Pogo Pad" x="13.46" y="23" rot="MR0"/>
-<element name="J3" library="SparkFun-Connectors" package="PAD.03X.03" value="Pogo Pad" x="16" y="20.46" rot="MR0"/>
-<element name="J4" library="SparkFun-Connectors" package="PAD.03X.03" value="Pogo Pad" x="13.46" y="20.46" rot="MR0"/>
-<element name="J5" library="SparkFun-Connectors" package="PAD.03X.03" value="Pogo Pad" x="16" y="17.92" rot="MR0"/>
-<element name="J6" library="SparkFun-Connectors" package="PAD.03X.03" value="Pogo Pad" x="13.46" y="17.92" rot="MR0"/>
+<element name="H2" library="holes" library_urn="urn:adsk.eagle:library:237" package="4,3-PAD" value="Mounting Pad" x="7.5" y="6" smashed="yes"/>
+<element name="J1" library="SparkFun-Connectors" package="PAD.03X.03" value="Pogo Pad" x="16" y="23" smashed="yes" rot="MR0"/>
+<element name="J2" library="SparkFun-Connectors" package="PAD.03X.03" value="Pogo Pad" x="13.46" y="23" smashed="yes" rot="MR0"/>
+<element name="J3" library="SparkFun-Connectors" package="PAD.03X.03" value="Pogo Pad" x="16" y="20.46" smashed="yes" rot="MR0"/>
+<element name="J4" library="SparkFun-Connectors" package="PAD.03X.03" value="Pogo Pad" x="13.46" y="20.46" smashed="yes" rot="MR0"/>
+<element name="J5" library="SparkFun-Connectors" package="PAD.03X.03" value="Pogo Pad" x="16" y="17.92" smashed="yes" rot="MR0"/>
+<element name="J6" library="SparkFun-Connectors" package="PAD.03X.03" value="Pogo Pad" x="13.46" y="17.92" smashed="yes" rot="MR0"/>
 </elements>
 <signals>
@@
 <wire x1="13.46" y1="17.92" x2="12.5" y2="16.96" width="0.36" layer="16"/>
 <wire x1="12.5" y1="16.96" x2="12.5" y2="16.5" width="0.36" layer="16"/>
+<via x="3.67" y="22.94" extent="1-16" drill="0.35"/>
+<polygon width="0.1524" layer="1" isolate="0.4" thermals="no">
+<vertex x="6" y="11"/>
+<vertex x="10" y="11"/>
+<vertex x="12.5" y="8.5"/>
+<vertex x="12.5" y="3.5"/>
+<vertex x="9.5" y="0.5"/>
+<vertex x="5" y="0.5"/>
+<vertex x="2" y="3.5"/>
+<vertex x="2" y="9"/>
+<vertex x="4" y="11"/>
+</polygon>
+<polygon width="0.1524" layer="1" thermals="no">
+<vertex x="0.5" y="25"/>
+<vertex x="12.5" y="25"/>
+<vertex x="12.5" y="21.3"/>
+<vertex x="0.5" y="21.3"/>
+</polygon>
+<polygon width="0.1524" layer="16" isolate="0.4" thermals="no" rank="2">
+<vertex x="0.5" y="25"/>
+<vertex x="10.5" y="25"/>
+<vertex x="10.5" y="21"/>
+<vertex x="0.5" y="21"/>
+</polygon>
+<via x="9.02" y="22.94" extent="1-16" drill="0.35"/>
 </signal>
 <signal name="VCC">
 <contactref element="C1" pad="1"/>
 <contactref element="R4" pad="2"/>
-<polygon width="0.1524" layer="16" isolate="0.4" thermals="no">
-<vertex x="0.5" y="25"/>
-<vertex x="21" y="25"/>
-<vertex x="21" y="0.5"/>
-<vertex x="0.5" y="0.5"/>
-</polygon>
 <contactref element="U1" pad="8"/>
 <contactref element="R6" pad="2"/>
@@
 <wire x1="19.405" y1="7.346" x2="19.405" y2="9.405" width="0.56" layer="1"/>
 <wire x1="19.405" y1="9.405" x2="19.5" y2="9.5" width="0.56" layer="1"/>
+<polygon width="0.1524" layer="16" isolate="0.4" thermals="no">
+<vertex x="0.5" y="21"/>
+<vertex x="10.5" y="21"/>
+<vertex x="10.5" y="25"/>
+<vertex x="21" y="25"/>
+<vertex x="21" y="0.5"/>
+<vertex x="0.5" y="0.5"/>
+</polygon>
 </signal>
 <signal name="D-">
@@
 </signal>
 </signals>
+<mfgpreviewcolors>
+<mfgpreviewcolor name="soldermaskcolor" color="0xC8008000"/>
+<mfgpreviewcolor name="silkscreencolor" color="0xFFFEFEFE"/>
+<mfgpreviewcolor name="backgroundcolor" color="0xFF282828"/>
+<mfgpreviewcolor name="coppercolor" color="0xFFFFBF00"/>
+<mfgpreviewcolor name="substratecolor" color="0xFF786E46"/>
+</mfgpreviewcolors>
 <errors>
 </errors>
@@
 <compatibility>
 <note version="8.2" severity="warning">
-Since Version 8.2, Eagle supports online libraries. The ids
+Since Version 8.2, EAGLE supports online libraries. The ids
 of those online libraries will not be understood (or retained)
 with this version.
